File: PCB_Frequency-meter-based-on-STM32/Shield_Frequency_meter_STM32/Shield_Frequency_meter_STM32.kicad_pcb (KiCad board)
At the start: 4 copper layers, 57.6 x 53.3 mm, 24 parts, among them J1 Power, J2 Digital/PWM, J3 Analog, J4 Digital/PWM, J5 +5V_PWR, J6 +5V_EXT, J7 Conn_Coaxial, U1 TPS60401DBV, U2 OPA210

Commit message: final PCB update
Parts:
- added C6: 22p, Capacitor_SMD:C_0603_1608Metric_Pad1.08x0.95mm_HandSolder, F.Cu at (151.2, 53.9)
- added C7: 47p, Capacitor_SMD:C_0805_2012Metric_Pad1.18x1.45mm_HandSolder, F.Cu at (153.6, 53.8)
- added C8: 0.1uF, Capacitor_SMD:C_1206_3216Metric_Pad1.33x1.80mm_HandSolder, F.Cu at (153.2, 63.2)
- added J10: Conn_01x01, Connector_PinHeader_2.54mm:PinHeader_1x01_P2.54mm_Vertical, F.Cu at (150.2, 71.2)
- added J8: Conn_01x01, Connector_PinHeader_2.54mm:PinHeader_1x01_P2.54mm_Vertical, F.Cu at (137.0, 53.6)
- added J9: Conn_01x01, Connector_PinHeader_2.54mm:PinHeader_1x01_P2.54mm_Vertical, F.Cu at (137.0, 62.4)
- moved R2 9.82 mm to (147.7, 59.9), turned to 180 degrees
- moved R3 4.16 mm to (147.7, 62.3), turned to 0 degrees
- moved C2 3.99 mm to (145.2, 86.0)
- moved C1 3.91 mm to (136.0, 86.7)
- moved C5 3.87 mm to (149.2, 54.6), turned to -90 degrees
- moved U1 3.86 mm to (140.1, 85.6)
- moved C3 3.26 mm to (140.2, 81.0)
- moved C4 3.22 mm to (143.0, 67.6)
- moved R1 3.22 mm to (139.2, 67.0)
- moved J5 2.55 mm to (128.1, 90.5)
- moved U2 2.04 mm to (148.2, 66.0)
- moved R5 0.70 mm to (145.8, 54.2)
- moved R4 0.47 mm to (142.8, 54.2), turned to 90 degrees
- moved D1 0.40 mm to (142.1, 59.4), turned to 180 degrees
Routing:
- net GND: track 0.00 -> 25.4 mm, vias 0 -> 7
- net /7: track 7.20 -> 21.7 mm
- net Net-(J9-Pin_1): track 8.66 -> 14.6 mm
- net -5V: track 11.1 -> 7.34 mm, vias 2 -> 0
- net /+5V_STM: track 11.2 -> 14.3 mm
- net +5V: track 50.3 -> 47.5 mm
- net Net-(U2-+In): track 6.38 -> 8.53 mm
- net Net-(D1-Pad3): track 4.11 -> 5.78 mm
- net Net-(U1-OUT): track 15.5 -> 16.9 mm
- removed copper zone on F.Cu, net GND
Other:
- copper layers 4 -> 2
- rule pad_to_mask_clearance: 0 -> 0.038
- board text added: "+"
- board text added: "-"
- board text added: "RECT_SIG_3.3"
- board text added: "RECT_SIG_5"
- board text added: "SIG_IN"
