File: PCB_Frequency-meter-based-on-STM32/Shield_Frequency_meter_STM32/Shield_Frequency_meter_STM32.kicad_sch (KiCad schematic)
At the start: 20 parts, among them J1 Power, J2 Digital/PWM, J3 Analog, J4 Digital/PWM, J5 +5V_PWR, J6 +5V_EXT, J7 Conn_Coaxial, U1 TPS60401DBV, U2 OPA210

Commit message: final PCB update
Parts:
- added C6: 22p, Capacitor_SMD:C_0603_1608Metric_Pad1.08x0.95mm_HandSolder, symbol Device:C
- added C7: 47p, Capacitor_SMD:C_0805_2012Metric_Pad1.18x1.45mm_HandSolder, symbol Device:C
- added C8: 0.1uF, Capacitor_SMD:C_1206_3216Metric_Pad1.33x1.80mm_HandSolder, symbol Shield_Frequency_meter:C1206C474J5NACTU
- added J10, J8, J9: Conn_01x01, Connector_PinHeader_2.54mm:PinHeader_1x01_P2.54mm_Vertical, symbol Connector_Generic:Conn_01x01
Connections:
- net +5V: now also C8.1
- net 7: now also C6.1, C7.1, J8.1 (Pin_1)
- net GND: now also C6.2, C7.2, C8.2
- net SIG_IN: now also J10.1 (Pin_1)
- net at D1.1, R3.1, U2.1 (Out): now also J9.1 (Pin_1)
